Commit message: Remove dae meshes from collision and add stl meshes instead

File: ur_description/urdf/ur10.urdf.xacro (robot description, xacro)
@@ -62,5 +62,5 @@
       <collision>
         <geometry>
-          <mesh filename="package://ur_description/meshes/ur10/collision/Base.dae"/>
+          <mesh filename="package://ur_description/meshes/ur10/collision/base.stl"/>
         </geometry>
       </collision>
@@ -90,5 +90,5 @@
       <collision>
         <geometry>
-          <mesh filename="package://ur_description/meshes/ur10/collision/Shoulder.dae"/>
+          <mesh filename="package://ur_description/meshes/ur10/collision/shoulder.stl"/>
         </geometry>
       </collision>
@@ -118,5 +118,5 @@
       <collision>
         <geometry>
-          <mesh filename="package://ur_description/meshes/ur10/collision/UpperArm.dae"/>
+          <mesh filename="package://ur_description/meshes/ur10/collision/upper_arm.stl"/>
         </geometry>
       </collision>
@@ -146,5 +146,5 @@
       <collision>
         <geometry>
-          <mesh filename="package://ur_description/meshes/ur10/collision/Forearm.dae"/>
+          <mesh filename="package://ur_description/meshes/ur10/collision/forearm.stl"/>
         </geometry>
       </collision>
@@ -174,5 +174,5 @@
       <collision>
         <geometry>
-          <mesh filename="package://ur_description/meshes/ur10/collision/Wrist1.dae"/>
+          <mesh filename="package://ur_description/meshes/ur10/collision/wrist_1.stl"/>
         </geometry>
       </collision>
@@ -202,5 +202,5 @@
       <collision>
         <geometry>
-          <mesh filename="package://ur_description/meshes/ur10/collision/Wrist2.dae"/>
+          <mesh filename="package://ur_description/meshes/ur10/collision/wrist_2.stl"/>
         </geometry>
       </collision>
@@ -230,5 +230,5 @@
       <collision>
         <geometry>
-          <mesh filename="package://ur_description/meshes/ur10/collision/Wrist3.dae"/>
+          <mesh filename="package://ur_description/meshes/ur10/collision/wrist_3.stl"/>
         </geometry>
       </collision>
@@ -242,5 +242,12 @@
       <origin xyz="0.0 ${wrist_3_length} 0.0" rpy="0.0 0.0 ${pi/2.0}" />
     </joint>
-    <link name="${prefix}ee_link" />
+    <link name="${prefix}ee_link">
+      <collision>
+        <geometry>
+          <box size="0.01 0.01 0.01"/>
+        </geometry>
+        <origin rpy="0 0 0" xyz="-0.01 0 0"/>
+      </collision>
+    </link>
     <xacro:ur10_arm_transmission prefix="${prefix}" />
     <xacro:ur10_arm_gazebo prefix="${prefix}" />
